Commit message: Created the forward kinematics

File: src/rrbot_description/urdf/rrbot.xacro (robot description, xacro)
@@ -143,3 +143,9 @@
     </inertial>
   </link>
+  <joint name="end_effector_joint" type="fixed">
+    <parent link="link3"/>
+    <child link="end_effector"/>
+    <origin xyz="0.0 0.0 ${height3 - axel_offset}" rpy="0.0 0.0 0.0"/>
+  </joint>
+  <link name="end_effector"/>
 </robot>
